File: motor_board.kicad_pcb (KiCad board)
At the start: 2 copper layers, 66 x 50 mm, 45 parts, among them J1 AUX1, J10 SERVO1, J11 SERVO2, J12 DEBUG, J13 RS485, J2 AUX2, J3 Conn_01x15, J4 MOTOR, J5 AUX3, J6 AUX4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

Commit message: Updated to KiCad 6
Other:
- net class Default removed
- board text added: "MOTOR DRIVER INTERFACE BOARD FOR USE WITH ST EV-VNH7070AS DESIGNED FOR MOTORS UP TO 4A STALL CURRENT."
- board text removed: "MOTOR DRIVER INTERFACE BOARD FOR USE WITH ST EV-VNH7070AS DESIGNED FOR MOTORS UP TO 4A STALL CURRENT. https://nathandumont.com/blog/robot-motor-control-board"
